Commit message: modified:   examples/agents/dart_cloth_agent_test.py 	modified:   gym/envs/__init__.py 	modified:   gym/envs/dart/__init__.py 	modified:   gym/envs/dart/assets/sawyer_description/urdf/sawyer_arm_hoop.urdf 	modified:   gym/envs/dart/upperbodydatadriven_cloth_base.py 	modified:   gym/envs/dart/upperbodydatadriven_rigidcloth_sawyer.py 	new file:   gym/envs/dart/upperbodydatadriven_rigidclothconstruct_sawyer.py 	new file:   gym/envs/dart/upperbodydatadriven_rigidclothhang_sawyer.py

File: gym/envs/dart/assets/sawyer_description/urdf/sawyer_arm_hoop.urdf (robot description, URDF)
Before this commit: robot sawyer, 20 links, 19 joints
Joints:
- joint right_hoop_j2: origin xyz=0 0 0.0245 rpy=0 0 0 -> xyz=0 0 0 rpy=0 0 0; parent right_hand -> right_hoop_1
- joint right_hoop_j3: origin xyz=0 0 0.0245 rpy=0 0 0 -> xyz=0 0 0 rpy=0 0 0; parent right_hand -> right_hoop_1
- joint right_hoop_j4: origin xyz=0 0 0.0245 rpy=0 0 0 -> xyz=0 0 0 rpy=0 0 0; parent right_hand -> right_hoop_1
