Commit message: modified:   examples/agents/dart_cloth_agent_test.py 	modified:   gym/envs/__init__.py 	modified:   gym/envs/dart/__init__.py 	modified:   gym/envs/dart/assets/sawyer_description/urdf/hoop_weldhang.urdf 	modified:   gym/envs/dart/static_cloth_window.py 	modified:   gym/envs/dart/upperbodydatadriven_cloth_base.py 	modified:   gym/envs/dart/upperbodydatadriven_rigidclothconstruct_sawyer.py 	new file:   gym/envs/dart/upperbodydatadriven_rigidclothonefile_sawyer.py

File: gym/envs/dart/assets/sawyer_description/urdf/hoop_weldhang.urdf (robot description, URDF)
Before this commit: robot hoop, 7 links, 6 joints
Joints:
- joint right_hoop_dj1: axis 0 1 0 -> 0 0 1; origin xyz=0 0 0.05 rpy=0 0 0 -> xyz=0 0 0.05 rpy=1.56 0 0
- joint right_hoop_dj2: axis 0 0 1 -> 0 1 0
