Commit message: modified:   gym/envs/dart/assets/iiwa_description/urdf/iiwa7_simplified.urdf

File: gym/envs/dart/assets/iiwa_description/urdf/iiwa7_simplified.urdf (robot description, URDF)
Before this commit: robot iiwa7, 10 links, 9 joints
Links:
- link iiwa_link_0: geometry visual mesh filename=../meshes/iiwa7/visual/link_0.stl
