Commit message: update walk keyframe motion

File: gym/envs/dart/assets/darwinmodel/coord.urdf (robot description, URDF)
Before this commit: robot coord, 4 links, 3 joints
Links:
- link coord_x: geometry visual box size=0.25 0.005 0.005
- link coord_y: geometry visual box size=0.005 0.25 0.005
- link coord_z: geometry visual box size=0.005 0.005 0.25
