Commit message: update darwin

File: gym/envs/dart/assets/darwinmodel/ground1.urdf (robot description, URDF)
Before this commit: robot ground_skeleton, 2 links, 1 joints
Links:
- added link pillar1, mass 1.0; visual box size=0.1 0.1 10.0
- added link pillar2, mass 1.0; visual box size=0.1 0.1 10.0
- added link pillar3, mass 1.0; visual box size=0.1 0.1 10.0
Joints:
- added joint pillar1joint: type fixed, parent ground_link, child pillar1, origin xyz=0 0 0 rpy=0 0 0
- added joint pillar2joint: type fixed, parent ground_link, child pillar2, origin xyz=0 0 0 rpy=0 0 0
- added joint pillar3joint: type fixed, parent ground_link, child pillar3, origin xyz=0 0 0 rpy=0 0 0

Commit message: fix joint limit issue in dartwin

File: gym/envs/dart/assets/darwinmodel/ground1.urdf (robot description, URDF)
Before this commit: robot ground_skeleton, 5 links, 4 joints
Links:
- link ground_link: geometry collision box size=25 25 2.05; visual box size=25 25 2.05

Commit message: add step keyframe

File: gym/envs/dart/assets/darwinmodel/ground1.urdf (robot description, URDF)
Before this commit: robot ground_skeleton, 5 links, 4 joints
Links:
- link ground_link: geometry collision box size=125 25 2.05; visual box size=125 25 2.05

Commit message: update darwin

File: gym/envs/dart/assets/darwinmodel/ground1.urdf (robot description, URDF)
Before this commit: robot ground_skeleton, 5 links, 4 joints
Links:
- added link ground_link2, mass 1.0; collision box size=0.4 25 2.05; visual box size=0.4 25 2.05
Joints:
- added joint ground_joint2: type fixed, parent ground_link, child ground_link2, origin xyz=0 0 0 rpy=0 0 0
